File: ATTiny412/ATTiny412.kicad_pcb (KiCad board)
At the start: 2 copper layers, 18 x 24.3 mm, 27 parts, among them J1 Conn_01x04, J2 Conn_01x02, J3 Conn_01x04, U1 AP2204K-ADJ

Commit message: Silkscreens Updated and Board Outlines aligned
Other:
- board text added: "Development Board for the ATTiny412"
- board text removed: "Development Board for the ATTiny402"
Changed lines of the file:
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@@
     (35 F.Paste user hide)
     (36 B.SilkS user)
-    (37 F.SilkS user hide)
+    (37 F.SilkS user)
     (38 B.Mask user hide)
     (39 F.Mask user hide)
-    (40 Dwgs.User user hide)
+    (40 Dwgs.User user)
     (41 Cmts.User user hide)
     (42 Eco1.User user hide)
@@
       (xy -0.412988 -1.250149) (xy -0.204738 -1.25021) (xy 0.004564 -1.250214) (xy 0.213903 -1.250163)) (layer F.SilkS) (width 0.01))
   )
-  (gr_text "Development Board\nfor the ATTiny402" (at 169.545 114.046) (layer B.SilkS)
+  (gr_text "Development Board\nfor the ATTiny412" (at 169.545 114.046) (layer B.SilkS)
     (effects (font (size 0.7 0.8) (thickness 0.13)) (justify mirror))
   )
@@
   (dimension 10.16 (width 0.15) (layer Dwgs.User)
     (gr_text "10.160 mm" (at 156.1292 119.2276 90) (layer Dwgs.User)
-      (effects (font (size 1 1) (thickness 0.15)))
+      (effects (font (size 1 1) (thickness 0.15)) hide)
     )
     (feature1 (pts (xy 161.8742 114.1476) (xy 156.842779 114.1476)))
@@
   (dimension 19.177 (width 0.15) (layer Dwgs.User)
     (gr_text "19.177 mm" (at 152.9542 119.7991 90) (layer Dwgs.User)
-      (effects (font (size 1 1) (thickness 0.15)))
+      (effects (font (size 1 1) (thickness 0.15)) hide)
     )
     (feature1 (pts (xy 163.0172 110.2106) (xy 153.667779 110.2106)))
@@
   (dimension 24.257 (width 0.15) (layer Dwgs.User)
     (gr_text "24.257 mm" (at 150.0332 119.7991 90) (layer Dwgs.User)
-      (effects (font (size 1 1) (thickness 0.15)))
+      (effects (font (size 1 1) (thickness 0.15)) hide)
     )
     (feature1 (pts (xy 163.0172 107.6706) (xy 150.746779 107.6706)))
@@
   (dimension 12.954 (width 0.15) (layer Dwgs.User)
     (gr_text "12.954 mm" (at 169.4942 134.7516) (layer Dwgs.User)
-      (effects (font (size 1 1) (thickness 0.15)))
+      (effects (font (size 1 1) (thickness 0.15)) hide)
     )
     (feature1 (pts (xy 163.0172 129.3876) (xy 163.0172 134.038021)))
@@
   (dimension 15.24 (width 0.15) (layer Dwgs.User)
     (gr_text "15.240 mm" (at 169.4942 137.7996) (layer Dwgs.User)
-      (effects (font (size 1 1) (thickness 0.15)))
+      (effects (font (size 1 1) (thickness 0.15)) hide)
     )
     (feature1 (pts (xy 161.8742 124.3076) (xy 161.8742 137.086021)))
@@
   (dimension 18.034 (width 0.15) (layer Dwgs.User)
     (gr_text "18.034 mm" (at 169.4942 140.5936) (layer Dwgs.User)
-      (effects (font (size 1 1) (thickness 0.15)))
+      (effects (font (size 1 1) (thickness 0.15)) hide)
     )
     (feature1 (pts (xy 160.4772 129.3876) (xy 160.4772 139.880021)))
