File: ATTinyX12/ATTinyX12.kicad_pcb (KiCad board)
At the start: 2 copper layers, 17.8 x 22.9 mm, 27 parts, among them J1 Conn_01x05, J2 Conn_01x05, J4 UPDI, U1 AP7365

Commit message: ATTiny X12, X14 Silkscreen Revision
Parts:
- G***: footprint logo:logo54x76 -> logo:logo47x67
- moved G*** 4.33 mm to (62.9, 36.8)
- moved G*** 1.52 mm to (67.2, 36.8)
Other:
- board text added: "ATTiny214"
- board text added: "ATTiny414"
- board text removed: "NC"
- board text removed: "UPDI"
- board text removed: "www.SirBoard.com"
