File: ATTinyX14/ATTinyX14.kicad_pcb (KiCad board)
At the start: 2 copper layers, 30.5 x 17.8 mm, 30 parts, among them J1 Conn_01x08, J2 Conn_01x08, J4 UPDI, U1 AP7365

Commit message: ATTiny X12, X14 Silkscreen Revision
Parts:
- removed the G*** at (70.4, 37.0)
- G***: footprint logo:logo76x107 -> logo:logo63x89
- moved G*** 4.01 mm to (63.1, 37.0)
Other:
- board text added: "ATTiny1614"
- board text added: "ATTiny214"
- board text added: "ATTiny414"
- board text added: "ATTiny814"
- board text added: "UPDI"
